Commit message: working version dont want to lose lol

File: src/my_robot_description/urdf/robot_v2.xacro (robot description, xacro)
@@ -795,5 +795,5 @@
   <link name="wheel2">
     <inertial>
-      <origin xyz="0.100026 0.05775 -0.0195" rpy="1.5708 0 1.0472"/>
+      <origin xyz="0 0 -0.025" rpy="0 0 2.0944"/>  <!-- 120° -->
       <mass value="0.056156"/>
       <inertia ixx="1.10674e-05" iyy="1.10674e-05" izz="1.62852e-05"
@@ -801,5 +801,5 @@
     </inertial>
     <visual>
-      <origin xyz="0 0 -0.025" rpy="0 0 0"/>
+      <origin xyz="0 0 -0.025" rpy="0 0 2.0944"/>  <!-- 120° -->
       <geometry>
         <mesh filename="model://delivery_bot/meshes/wheel.stl"/>
@@ -807,5 +807,5 @@
     </visual>
     <collision>
-      <origin xyz="0 0 -0.025" rpy="0 0 0"/>
+      <origin xyz="0 0 -0.025" rpy="0 0 2.0944"/>  <!-- 120° -->
       <geometry>
         <mesh filename="model://delivery_bot/meshes/wheel.stl"/>
@@ -814,6 +814,5 @@
   </link>
   <joint name="wheel2_joint" type="revolute">
-    <origin xyz="0.100026 0.05775 -0.0195"
-            rpy="1.5708 0 0"/>
+     <origin xyz="0.100026 0.05775 -0.0195" rpy="1.5708 0 2.0944"/>
     <parent link="base_link"/>
     <child  link="wheel2"/>
@@ -835,5 +834,5 @@
   <link name="wheel3">
     <inertial>
-      <origin xyz="-0.100026 0.05775 -0.0195" rpy="1.5708 0 2.0944"/>
+      <origin xyz="0 0 -0.025" rpy="0 0 4.1888"/>  <!-- 240° -->
       <mass value="0.056156"/>
       <inertia ixx="1.10674e-05" iyy="1.10674e-05" izz="1.62852e-05"
@@ -841,5 +840,5 @@
     </inertial>
     <visual>
-      <origin xyz="0 0 -0.025" rpy="0 0 0"/>
+      <origin xyz="0 0 -0.025" rpy="0 0 4.1888"/>  <!-- 240° -->
       <geometry>
         <mesh filename="model://delivery_bot/meshes/wheel.stl"/>
@@ -847,5 +846,5 @@
     </visual>
     <collision>
-      <origin xyz="0 0 -0.025" rpy="0 0 0"/>
+      <origin xyz="0 0 -0.025" rpy="0 0 4.1888"/>  <!-- 240° -->
       <geometry>
         <mesh filename="model://delivery_bot/meshes/wheel.stl"/>
@@ -854,6 +853,5 @@
   </link>
   <joint name="wheel3_joint" type="revolute">
-    <origin xyz="-0.100026 0.05775 -0.0195"
-            rpy="1.5708 0 0"/>
+    <origin xyz="-0.100026 0.05775 -0.0195" rpy="1.5708 0 4.1888"/>
     <parent link="base_link"/>
     <child  link="wheel3"/>
