Commit message: ...

File: src/my_robot_description/urdf/robot_v3.xacro (robot description, xacro)
@@ -1,5 +1,3 @@
 <?xml version="1.0" ?>
-<!-- Generated using onshape-to-robot -->
-<!-- Onshape https://cad.onshape.com/documents/78378c45b2a0fb18e8081503/w/c19beaeea10b51c03146c067/e/4c0c92ba02de8a9d67d7ed4d -->
 <robot xmlns:xacro="http://www.ros.org/wiki/xacro" name="delivery_bot">
   <link name="base_link">
@@ -13,5 +11,5 @@
       <origin xyz="-0.0513068 -0.08 0.126" rpy="3.14159 -0 0"/>
       <geometry>
-        <mesh filename="model://delivery_bot/meshes//column_support.stl"/>
+        <mesh filename="file://$(find my_robot_description)/models/delivery_bot/meshes/column_support.stl"/>
       </geometry>
       <material name="column_support_material">
@@ -22,5 +20,5 @@
       <origin xyz="-0.0513068 -0.08 0.126" rpy="3.14159 -0 0"/>
       <geometry>
-        <mesh filename="model://delivery_bot/meshes//column_support.stl"/>
+        <mesh filename="file://$(find my_robot_description)/models/delivery_bot/meshes/column_support.stl"/>
       </geometry>
     </collision>
@@ -29,5 +27,5 @@
       <origin xyz="0.0436286 0.084433 0.006" rpy="0 -0 0"/>
       <geometry>
-        <mesh filename="model://delivery_bot/meshes//column_support.stl"/>
+        <mesh filename="file://$(find my_robot_description)/models/delivery_bot/meshes/column_support.stl"/>
       </geometry>
       <material name="column_support_2_material">
@@ -38,5 +36,5 @@
       <origin xyz="0.0436286 0.084433 0.006" rpy="0 -0 0"/>
       <geometry>
-        <mesh filename="model://delivery_bot/meshes//column_support.stl"/>
+        <mesh filename="file://$(find my_robot_description)/models/delivery_bot/meshes/column_support.stl"/>
       </geometry>
     </collision>
@@ -45,5 +43,5 @@
       <origin xyz="4.16334e-17 -0.12125 -0.0195" rpy="2.0506e-16 4.64408e-16 1.94289e-16"/>
       <geometry>
-        <mesh filename="model://delivery_bot/meshes//geared_dc_motor_with_encoder___ts_25ga370h.stl"/>
+        <mesh filename="file://$(find my_robot_description)/models/delivery_bot/meshes/geared_dc_motor_with_encoder___ts_25ga370h.stl"/>
       </geometry>
       <material name="geared_dc_motor_with_encoder___ts_25ga370h_material">
@@ -54,5 +52,5 @@
       <origin xyz="4.16334e-17 -0.12125 -0.0195" rpy="2.0506e-16 4.64408e-16 1.94289e-16"/>
       <geometry>
-        <mesh filename="model://delivery_bot/meshes//geared_dc_motor_with_encoder___ts_25ga370h.stl"/>
+        <mesh filename="file://$(find my_robot_description)/models/delivery_bot/meshes/geared_dc_motor_with_encoder___ts_25ga370h.stl"/>
       </geometry>
     </collision>
@@ -61,5 +59,5 @@
       <origin xyz="-0.105006 0.060625 -0.0195" rpy="-3.14159 4.27106e-44 1.0472"/>
       <geometry>
-        <mesh filename="model://delivery_bot/meshes//geared_dc_motor_with_encoder___ts_25ga370h.stl"/>
+        <mesh filename="file://$(find my_robot_description)/models/delivery_bot/meshes/geared_dc_motor_with_encoder___ts_25ga370h.stl"/>
       </geometry>
       <material name="geared_dc_motor_with_encoder___ts_25ga370h_2_material">
@@ -70,5 +68,5 @@
       <origin xyz="-0.105006 0.060625 -0.0195" rpy="-3.14159 4.27106e-44 1.0472"/>
       <geometry>
-        <mesh filename="model://delivery_bot/meshes//geared_dc_motor_with_encoder___ts_25ga370h.stl"/>
+        <mesh filename="file://$(find my_robot_description)/models/delivery_bot/meshes/geared_dc_motor_with_encoder___ts_25ga370h.stl"/>
       </geometry>
     </collision>
@@ -77,5 +75,5 @@
       <origin xyz="3.46945e-17 -0.08 0" rpy="-3.14159 4.64408e-16 1.94289e-16"/>
       <geometry>
-        <mesh filename="model://delivery_bot/meshes//motor_mount.stl"/>
+        <mesh filename="file://$(find my_robot_description)/models/delivery_bot/meshes/motor_mount.stl"/>
       </geometry>
       <material name="motor_mount_material">
@@ -86,5 +84,5 @@
       <origin xyz="3.46945e-17 -0.08 0" rpy="-3.14159 4.64408e-16 1.94289e-16"/>
       <geometry>
-        <mesh filename="model://delivery_bot/meshes//motor_mount.stl"/>
+        <mesh filename="file://$(find my_robot_description)/models/delivery_bot/meshes/motor_mount.stl"/>
       </geometry>
     </collision>
@@ -93,5 +91,5 @@
       <origin xyz="0.105006 0.060625 -0.0195" rpy="3.14159 5.47382e-48 -1.0472"/>
       <geometry>
-        <mesh filename="model://delivery_bot/meshes//geared_dc_motor_with_encoder___ts_25ga370h.stl"/>
+        <mesh filename="file://$(find my_robot_description)/models/delivery_bot/meshes/geared_dc_motor_with_encoder___ts_25ga370h.stl"/>
       </geometry>
       <material name="geared_dc_motor_with_encoder___ts_25ga370h_3_material">
@@ -102,5 +100,5 @@
       <origin xyz="0.105006 0.060625 -0.0195" rpy="3.14159 5.47382e-48 -1.0472"/>
       <geometry>
-        <mesh filename="model://delivery_bot/meshes//geared_dc_motor_with_encoder___ts_25ga370h.stl"/>
+        <mesh filename="file://$(find my_robot_description)/models/delivery_bot/meshes/geared_dc_motor_with_encoder___ts_25ga370h.stl"/>
       </geometry>
     </collision>
@@ -109,5 +107,5 @@
       <origin xyz="-0.0436286 0.084433 0.126" rpy="3.14159 -0 0"/>
       <geometry>
-        <mesh filename="model://delivery_bot/meshes//column_support.stl"/>
+        <mesh filename="file://$(find my_robot_description)/models/delivery_bot/meshes/column_support.stl"/>
       </geometry>
       <material name="column_support_3_material">
@@ -118,5 +116,5 @@
       <origin xyz="-0.0436286 0.084433 0.126" rpy="3.14159 -0 0"/>
       <geometry>
-        <mesh filename="model://delivery_bot/meshes//column_support.stl"/>
+        <mesh filename="file://$(find my_robot_description)/models/delivery_bot/meshes/column_support.stl"/>
       </geometry>
     </collision>
@@ -125,5 +123,5 @@
       <origin xyz="0.0513068 -0.08 0.126" rpy="3.14159 -0 0"/>
       <geometry>
-        <mesh filename="model://delivery_bot/meshes//column_support.stl"/>
+        <mesh filename="file://$(find my_robot_description)/models/delivery_bot/meshes/column_support.stl"/>
       </geometry>
       <material name="column_support_4_material">
@@ -134,5 +132,5 @@
       <origin xyz="0.0513068 -0.08 0.126" rpy="3.14159 -0 0"/>
       <geometry>
-        <mesh filename="model://delivery_bot/meshes//column_support.stl"/>
+        <mesh filename="file://$(find my_robot_description)/models/delivery_bot/meshes/column_support.stl"/>
       </geometry>
     </collision>
@@ -141,5 +139,5 @@
       <origin xyz="-0.0949354 -0.00443297 0.126" rpy="3.14159 -0 0"/>
       <geometry>
-        <mesh filename="model://delivery_bot/meshes//column_support.stl"/>
+        <mesh filename="file://$(find my_robot_description)/models/delivery_bot/meshes/column_support.stl"/>
       </geometry>
       <material name="column_support_5_material">
@@ -150,5 +148,5 @@
       <origin xyz="-0.0949354 -0.00443297 0.126" rpy="3.14159 -0 0"/>
       <geometry>
-        <mesh filename="model://delivery_bot/meshes//column_support.stl"/>
+        <mesh filename="file://$(find my_robot_description)/models/delivery_bot/meshes/column_support.stl"/>
       </geometry>
     </collision>
@@ -157,5 +155,5 @@
       <origin xyz="0 0 0" rpy="0 -0 0"/>
       <geometry>
-        <mesh filename="model://delivery_bot/meshes//base_link.stl"/>
+        <mesh filename="file://$(find my_robot_description)/models/delivery_bot/meshes/base_link.stl"/>
       </geometry>
       <material name="base_link_material">
@@ -166,5 +164,5 @@
       <origin xyz="0 0 0" rpy="0 -0 0"/>
       <geometry>
-        <mesh filename="model://delivery_bot/meshes//base_link.stl"/>
+        <mesh filename="file://$(find my_robot_description)/models/delivery_bot/meshes/base_link.stl"/>
       </geometry>
     </collision>
@@ -173,5 +171,5 @@
       <origin xyz="9.02056e-17 -1.38778e-17 0.132" rpy="3.14159 -0 3.14159"/>
       <geometry>
-        <mesh filename="model://delivery_bot/meshes//top_plate.stl"/>
+        <mesh filename="file://$(find my_robot_description)/models/delivery_bot/meshes/top_plate.stl"/>
       </geometry>
       <material name="top_plate_material">
@@ -182,5 +180,5 @@
       <origin xyz="9.02056e-17 -1.38778e-17 0.132" rpy="3.14159 -0 3.14159"/>
       <geometry>
-        <mesh filename="model://delivery_bot/meshes//top_plate.stl"/>
+        <mesh filename="file://$(find my_robot_description)/models/delivery_bot/meshes/top_plate.stl"/>
       </geometry>
     </collision>
@@ -189,5 +187,5 @@
       <origin xyz="-0.069282 0.04 -6.55569e-45" rpy="3.14159 -4.28639e-44 -2.0944"/>
       <geometry>
-        <mesh filename="model://delivery_bot/meshes//motor_mount.stl"/>
+        <mesh filename="file://$(find my_robot_description)/models/delivery_bot/meshes/motor_mount.stl"/>
       </geometry>
       <material name="motor_mount_2_material">
@@ -198,5 +196,5 @@
       <origin xyz="-0.069282 0.04 -6.55569e-45" rpy="3.14159 -4.28639e-44 -2.0944"/>
       <geometry>
-        <mesh filename="model://delivery_bot/meshes//motor_mount.stl"/>
+        <mesh filename="file://$(find my_robot_description)/models/delivery_bot/meshes/motor_mount.stl"/>
       </geometry>
     </collision>
@@ -205,5 +203,5 @@
       <origin xyz="0.069282 0.04 0" rpy="3.14159 3.61234e-97 2.0944"/>
       <geometry>
-        <mesh filename="model://delivery_bot/meshes//motor_mount.stl"/>
+        <mesh filename="file://$(find my_robot_description)/models/delivery_bot/meshes/motor_mount.stl"/>
       </geometry>
       <material name="motor_mount_3_material">
@@ -214,5 +212,5 @@
       <origin xyz="0.069282 0.04 0" rpy="3.14159 3.61234e-97 2.0944"/>
       <geometry>
-        <mesh filename="model://delivery_bot/meshes//motor_mount.stl"/>
+        <mesh filename="file://$(find my_robot_description)/models/delivery_bot/meshes/motor_mount.stl"/>
       </geometry>
     </collision>
@@ -221,5 +219,5 @@
       <origin xyz="0.0949354 -0.00443297 0.126" rpy="3.14159 -0 0"/>
       <geometry>
-        <mesh filename="model://delivery_bot/meshes//column_support.stl"/>
+        <mesh filename="file://$(find my_robot_description)/models/delivery_bot/meshes/column_support.stl"/>
       </geometry>
       <material name="column_support_6_material">
@@ -230,5 +228,5 @@
       <origin xyz="0.0949354 -0.00443297 0.126" rpy="3.14159 -0 0"/>
       <geometry>
-        <mesh filename="model://delivery_bot/meshes//column_support.stl"/>
+        <mesh filename="file://$(find my_robot_description)/models/delivery_bot/meshes/column_support.stl"/>
       </geometry>
     </collision>
@@ -237,5 +235,5 @@
       <origin xyz="-0.0121949 0.0322049 0.1791" rpy="-2.74517 1.5708 0"/>
       <geometry>
-        <mesh filename="model://delivery_bot/meshes//part_8.stl"/>
+        <mesh filename="file://$(find my_robot_description)/models/delivery_bot/meshes/part_8.stl"/>
       </geometry>
       <material name="part_8_material">
@@ -246,5 +244,5 @@
       <origin xyz="-0.0121949 0.0322049 0.1791" rpy="-2.74517 1.5708 0"/>
       <geometry>
-        <mesh filename="model://delivery_bot/meshes//part_8.stl"/>
+        <mesh filename="file://$(find my_robot_description)/models/delivery_bot/meshes/part_8.stl"/>
       </geometry>
     </collision>
@@ -253,5 +251,5 @@
       <origin xyz="-0.028 0.035 0.1416" rpy="0 -0 -1.5708"/>
       <geometry>
-        <mesh filename="model://delivery_bot/meshes//part_15.stl"/>
+        <mesh filename="file://$(find my_robot_description)/models/delivery_bot/meshes/part_15.stl"/>
       </geometry>
       <material name="part_15_material">
@@ -262,5 +260,5 @@
       <origin xyz="-0.028 0.035 0.1416" rpy="0 -0 -1.5708"/>
       <geometry>
-        <mesh filename="model://delivery_bot/meshes//part_15.stl"/>
+        <mesh filename="file://$(find my_robot_description)/models/delivery_bot/meshes/part_15.stl"/>
       </geometry>
     </collision>
@@ -269,5 +267,5 @@
       <origin xyz="-9.44383e-15 -0.0385 0.1411" rpy="-6.12279e-17 -6.12323e-17 -3.14159"/>
       <geometry>
-        <mesh filename="model://delivery_bot/meshes//part_11.stl"/>
+        <mesh filename="file://$(find my_robot_description)/models/delivery_bot/meshes/part_11.stl"/>
       </geometry>
       <material name="part_11_material">
@@ -278,5 +276,5 @@
       <origin xyz="-9.44383e-15 -0.0385 0.1411" rpy="-6.12279e-17 -6.12323e-17 -3.14159"/>
       <geometry>
-        <mesh filename="model://delivery_bot/meshes//part_11.stl"/>
+        <mesh filename="file://$(find my_robot_description)/models/delivery_bot/meshes/part_11.stl"/>
       </geometry>
     </collision>
@@ -285,5 +283,5 @@
       <origin xyz="-0.011 -0.0385 0.1629" rpy="1.53787 1.5708 0"/>
       <geometry>
-        <mesh filename="model://delivery_bot/meshes//part_8.stl"/>
+        <mesh filename="file://$(find my_robot_description)/models/delivery_bot/meshes/part_8.stl"/>
       </geometry>
       <material name="part_8_2_material">
@@ -294,5 +292,5 @@
       <origin xyz="-0.011 -0.0385 0.1629" rpy="1.53787 1.5708 0"/>
       <geometry>
-        <mesh filename="model://delivery_bot/meshes//part_8.stl"/>
+        <mesh filename="file://$(find my_robot_description)/models/delivery_bot/meshes/part_8.stl"/>
       </geometry>
     </collision>
@@ -301,5 +299,5 @@
       <origin xyz="-9.44383e-15 -0.0385 0.1616" rpy="1.28639e-16 3.79626e-17 0.124422"/>
       <geometry>
-        <mesh filename="model://delivery_bot/meshes//part_20.stl"/>
+        <mesh filename="file://$(find my_robot_description)/models/delivery_bot/meshes/part_20.stl"/>
       </geometry>
       <material name="part_20_material">
@@ -310,5 +308,5 @@
       <origin xyz="-9.44383e-15 -0.0385 0.1616" rpy="1.28639e-16 3.79626e-17 0.124422"/>
       <geometry>
-        <mesh filename="model://delivery_bot/meshes//part_20.stl"/>
+        <mesh filename="file://$(find my_robot_description)/models/delivery_bot/meshes/part_20.stl"/>
       </geometry>
     </collision>
@@ -317,5 +315,5 @@
       <origin xyz="0.02 -0.035 0.14" rpy="3.14159 -0 -1.5708"/>
       <geometry>
-        <mesh filename="model://delivery_bot/meshes//part_16.stl"/>
+        <mesh filename="file://$(find my_robot_description)/models/delivery_bot/meshes/part_16.stl"/>
       </geometry>
       <material name="part_16_material">
@@ -326,5 +324,5 @@
       <origin xyz="0.02 -0.035 0.14" rpy="3.14159 -0 -1.5708"/>
       <geometry>
-        <mesh filename="model://delivery_bot/meshes//part_16.stl"/>
+        <mesh filename="file://$(find my_robot_description)/models/delivery_bot/meshes/part_16.stl"/>
       </geometry>
     </collision>
@@ -333,5 +331,5 @@
       <origin xyz="-0.02 -0.035 0.14" rpy="3.14159 -0 -1.5708"/>
       <geometry>
-        <mesh filename="model://delivery_bot/meshes//part_16.stl"/>
+        <mesh filename="file://$(find my_robot_description)/models/delivery_bot/meshes/part_16.stl"/>
       </geometry>
       <material name="part_16_2_material">
@@ -342,5 +340,5 @@
       <origin xyz="-0.02 -0.035 0.14" rpy="3.14159 -0 -1.5708"/>
       <geometry>
-        <mesh filename="model://delivery_bot/meshes//part_16.stl"/>
+        <mesh filename="file://$(find my_robot_description)/models/delivery_bot/meshes/part_16.stl"/>
       </geometry>
     </collision>
@@ -349,5 +347,5 @@
       <origin xyz="-0.02 -0.035 0.1416" rpy="0 -0 -1.5708"/>
       <geometry>
-        <mesh filename="model://delivery_bot/meshes//part_15.stl"/>
+        <mesh filename="file://$(find my_robot_description)/models/delivery_bot/meshes/part_15.stl"/>
       </geometry>
       <material name="part_15_2_material">
@@ -358,5 +356,5 @@
       <origin xyz="-0.02 -0.035 0.1416" rpy="0 -0 -1.5708"/>
       <geometry>
-        <mesh filename="model://delivery_bot/meshes//part_15.stl"/>
+        <mesh filename="file://$(find my_robot_description)/models/delivery_bot/meshes/part_15.stl"/>
       </geometry>
     </collision>
@@ -365,5 +363,5 @@
       <origin xyz="-9.44383e-15 0.007 0.1606" rpy="0 -0 -1.5708"/>
       <geometry>
-        <mesh filename="model://delivery_bot/meshes//part_1.stl"/>
+        <mesh filename="file://$(find my_robot_description)/models/delivery_bot/meshes/part_1.stl"/>
       </geometry>
       <material name="part_1_material">
@@ -374,5 +372,5 @@
       <origin xyz="-9.44383e-15 0.007 0.1606" rpy="0 -0 -1.5708"/>
       <geometry>
-        <mesh filename="model://delivery_bot/meshes//part_1.stl"/>
+        <mesh filename="file://$(find my_robot_description)/models/delivery_bot/meshes/part_1.stl"/>
       </geometry>
     </collision>
@@ -381,5 +379,5 @@
       <origin xyz="0.000111026 0.00693466 0.1761" rpy="3.14159 5.29332e-14 0.450629"/>
       <geometry>
-        <mesh filename="model://delivery_bot/meshes//part_1__2.stl"/>
+        <mesh filename="file://$(find my_robot_description)/models/delivery_bot/meshes/part_1__2.stl"/>
       </geometry>
       <material name="part_1_2_material">
@@ -390,5 +388,5 @@
       <origin xyz="0.000111026 0.00693466 0.1761" rpy="3.14159 5.29332e-14 0.450629"/>
       <geometry>
-        <mesh filename="model://delivery_bot/meshes//part_1__2.stl"/>
+        <mesh filename="file://$(find my_robot_description)/models/delivery_bot/meshes/part_1__2.stl"/>
       </geometry>
     </collision>
@@ -397,5 +395,5 @@
       <origin xyz="-9.44383e-15 0.007 0.1416" rpy="3.14159 -0 -1.5708"/>
       <geometry>
-        <mesh filename="model://delivery_bot/meshes//part_18.stl"/>
+        <mesh filename="file://$(find my_robot_description)/models/delivery_bot/meshes/part_18.stl"/>
       </geometry>
       <material name="part_18_material">
@@ -406,5 +404,5 @@
       <origin xyz="-9.44383e-15 0.007 0.1416" rpy="3.14159 -0 -1.5708"/>
       <geometry>
-        <mesh filename="model://delivery_bot/meshes//part_18.stl"/>
+        <mesh filename="file://$(find my_robot_description)/models/delivery_bot/meshes/part_18.stl"/>
       </geometry>
     </collision>
@@ -413,5 +411,5 @@
       <origin xyz="0.000125 -0.0152 0.14875" rpy="-3.14159 -1.22465e-16 3.14159"/>
       <geometry>
-        <mesh filename="model://delivery_bot/meshes//part_13.stl"/>
+        <mesh filename="file://$(find my_robot_description)/models/delivery_bot/meshes/part_13.stl"/>
       </geometry>
       <material name="part_13_material">
@@ -422,5 +420,5 @@
       <origin xyz="0.000125 -0.0152 0.14875" rpy="-3.14159 -1.22465e-16 3.14159"/>
       <geometry>
-        <mesh filename="model://delivery_bot/meshes//part_13.stl"/>
+        <mesh filename="file://$(find my_robot_description)/models/delivery_bot/meshes/part_13.stl"/>
       </geometry>
     </collision>
@@ -429,5 +427,5 @@
       <origin xyz="0.000362495 -0.026 0.1358" rpy="1.5708 -8.69586e-17 -3.14159"/>
       <geometry>
-        <mesh filename="model://delivery_bot/meshes//part_10.stl"/>
+        <mesh filename="file://$(find my_robot_description)/models/delivery_bot/meshes/part_10.stl"/>
       </geometry>
       <material name="part_10_material">
@@ -438,5 +436,5 @@
       <origin xyz="0.000362495 -0.026 0.1358" rpy="1.5708 -8.69586e-17 -3.14159"/>
       <geometry>
-        <mesh filename="model://delivery_bot/meshes//part_10.stl"/>
+        <mesh filename="file://$(find my_robot_description)/models/delivery_bot/meshes/part_10.stl"/>
       </geometry>
     </collision>
@@ -445,5 +443,5 @@
       <origin xyz="0.011 -0.0385 0.1629" rpy="1.53787 1.5708 0"/>
       <geometry>
-        <mesh filename="model://delivery_bot/meshes//part_8.stl"/>
+        <mesh filename="file://$(find my_robot_description)/models/delivery_bot/meshes/part_8.stl"/>
       </geometry>
       <material name="part_8_3_material">
@@ -454,5 +452,5 @@
       <origin xyz="0.011 -0.0385 0.1629" rpy="1.53787 1.5708 0"/>
       <geometry>
-        <mesh filename="model://delivery_bot/meshes//part_8.stl"/>
+        <mesh filename="file://$(find my_robot_description)/models/delivery_bot/meshes/part_8.stl"/>
       </geometry>
     </collision>
@@ -461,5 +459,5 @@
       <origin xyz="-9.44383e-15 0.007 0.1496" rpy="0 -0 -1.5708"/>
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