Commit message: fixed control issues with omni drive controller

File: src/my_robot_description/urdf/robot_v3.xacro (robot description, xacro)
@@ -775,11 +775,15 @@
     </collision>
   </link>
-  <!-- Joint from base_link to wheel -->
-  <joint name="wheel1_joint" type="revolute">
+  <!-- wheel1: make it continuous and remove position limits -->
+  <joint name="wheel1_joint" type="continuous">
     <origin xyz="-0.100026 0.05775 -0.0195" rpy="1.5708 1.48832 1.0472"/>
     <parent link="base_link"/>
     <child link="wheel1"/>
+    <!-- Axis must be the wheel's spin axis in the JOINT frame -->
     <axis xyz="0 0 1"/>
-    <limit effort="10" velocity="10" lower="-3.141592653589793" upper="3.141592653589793"/>
+    <!-- Continuous joints ignore lower/upper. Keep effort/velocity. -->
+    <limit effort="5.0" velocity="100.0"/>
+    <!-- Helps kill jitter -->
+    <dynamics damping="0.2" friction="0.0"/>
   </joint>
   <!-- Link wheel2 -->
@@ -815,11 +819,15 @@
     </collision>
   </link>
-  <!-- Joint from base_link to wheel2 -->
-  <joint name="wheel2_joint" type="revolute">
+  <!-- wheel2: make it continuous and remove position limits -->
+  <joint name="wheel2_joint" type="continuous">
     <origin xyz="0.100026 0.05775 -0.0195" rpy="1.5708 -2.15704e-32 -1.0472"/>
     <parent link="base_link"/>
     <child link="wheel2"/>
+    <!-- Axis must be the wheel's spin axis in the JOINT frame -->
     <axis xyz="0 0 1"/>
-    <limit effort="10" velocity="10" lower="-3.141592653589793" upper="3.141592653589793"/>
+    <!-- Continuous joints ignore lower/upper. Keep effort/velocity. -->
+    <limit effort="5.0" velocity="100.0"/>
+    <!-- Helps kill jitter -->
+    <dynamics damping="0.2" friction="0.0"/>
   </joint>
   <!-- Link wheel3 -->
@@ -856,15 +864,20 @@
   </link>
   <!-- Joint from base_link to wheel3 -->
-  <joint name="wheel3_joint" type="revolute">
+<!-- wheel3: make it continuous and remove position limits -->
+  <joint name="wheel3_joint" type="continuous">
     <origin xyz="4.03566e-17 -0.1155 -0.0195" rpy="-1.5708 -2.04051e-15 2.22045e-16"/>
     <parent link="base_link"/>
     <child link="wheel3"/>
+    <!-- Axis must be the wheel's spin axis in the JOINT frame -->
     <axis xyz="0 0 1"/>
-    <limit effort="10" velocity="10" lower="-3.141592653589793" upper="3.141592653589793"/>
+    <!-- Continuous joints ignore lower/upper. Keep effort/velocity. -->
+    <limit effort="5.0" velocity="100.0"/>
+    <!-- Helps kill jitter -->
+    <dynamics damping="0.2" friction="0.0"/>
   </joint>
   <!-- ROS2 Control for Fortress -->
-  <ros2_control name="IgnitionSystem" type="system">
+  <ros2_control name="GazeboSimSystem" type="system">
     <hardware>
-      <plugin>ign_ros2_control/IgnitionSystem</plugin>
+      <plugin>gz_ros2_control/GazeboSimSystem</plugin>
     </hardware>
     <joint name="wheel1_joint">
@@ -890,5 +903,5 @@
       <robot_param>robot_description</robot_param>
       <robot_param_node>robot_state_publisher</robot_param_node>
-      <parameters>/home/abanoub/delivery_bot_ws/src/delivery_bot_control/config/gains.yaml</parameters>
+      <parameters>/home/abanoub/delivery_bot_ws/src/delivery_bot_control/config/omni_drive_controller.params.yaml</parameters>
     </plugin>
   </gazebo>

Commit message: added IMU support and EKF

File: src/my_robot_description/urdf/robot_v3.xacro (robot description, xacro)
@@ -1,4 +1,4 @@
 <?xml version="1.0" ?>
-<robot xmlns:xacro="http://www.ros.org/wiki/xacro" name="delivery_bot">
+<robot name="delivery_bot" xmlns:gz="http://gazebosim.org/schema">
   <link name="base_link">
     <inertial>
@@ -818,6 +818,5 @@
       </surface>
     </collision>
-  </link>
-  <!-- wheel2: make it continuous and remove position limits -->
+  </link>  <!-- wheel2: make it continuous and remove position limits -->
   <joint name="wheel2_joint" type="continuous">
     <origin xyz="0.100026 0.05775 -0.0195" rpy="1.5708 -2.15704e-32 -1.0472"/>
@@ -863,5 +862,5 @@
     </collision>
   </link>
-  <!-- Joint from base_link to wheel3 -->
+<!-- Joint from base_link to wheel3 -->
 <!-- wheel3: make it continuous and remove position limits -->
   <joint name="wheel3_joint" type="continuous">
@@ -907,8 +906,8 @@
   </gazebo>
   <gazebo reference="lidarView">
-      <sensor name="lidar_sensor" type="gpu_lidar">
+      <sensor name="lidarView" type="gpu_lidar">
           <pose>0 0 0 0 0 0</pose>
           <topic>lidar</topic>
-          <update_rate>10</update_rate>
+          <update_rate>20</update_rate>
           <ray>
             <scan>
@@ -936,3 +935,66 @@
         </sensor>
   </gazebo>
+  <!-- URDF file -->
+  <link name="imu_link">
+    <inertial><mass value="1e-6"/></inertial>
+  </link>
+  <joint name="imu_joint" type="fixed">
+    <parent link="base_link"/>
+    <child link="imu_link"/>
+    <origin xyz="0 0 0.10" rpy="0 0 0"/>
+  </joint>
+  <!-- SDF-in-URDF block that Gazebo reads -->
+  <gazebo reference="imu_link">
+    <sensor name="imu" type="imu">
+      <always_on>1</always_on>
+      <update_rate>100</update_rate>
+      <visualize>false</visualize>
+      <!-- Gazebo transport topic name; ros_gz_bridge will bridge this to ROS -->
+      <topic>imu</topic>
+      <!-- Frame id for ROS (supported by ros_gz); harmless warning if not recognized) -->
+      <gz_frame_id>imu_link</gz_frame_id>
+      <!-- Optional: add noise (example values) -->
+      <imu>
+      </imu>
+    </sensor>
+  </gazebo>
+    <!-- wheel1 -->
+  <gazebo reference="wheel1">
+    <mu1>1.6</mu1>
+    <mu2>0.01</mu2>
+    <!-- Try +X of wheel1 as rolling dir first -->
+    <fdir1 gz:expressed_in="wheel1">1 0 0</fdir1>
+  </gazebo>
+  <!-- wheel2 -->
+  <gazebo reference="wheel2">
+    <mu1>1.6</mu1>
+    <mu2>0.01</mu2>
+    <fdir1 gz:expressed_in="wheel2">0 1 0</fdir1>
+  </gazebo>
+  <!-- wheel3 -->
+  <gazebo reference="wheel3">
+    <mu1>1.6</mu1>
+    <mu2>0.01</mu2>
+    <fdir1 gz:expressed_in="wheel3">-1 0 0</fdir1>
+  </gazebo>
+  <gazebo>
+    <plugin name="ignition::gazebo::systems::WheelSlip"
+            filename="libignition-gazebo-wheel-slip-system.so">
+      <wheel link_name="wheel1">
+        <slip_compliance_lateral>0.05</slip_compliance_lateral>
+        <slip_compliance_longitudinal>0.0</slip_compliance_longitudinal>
+        <wheel_normal_force>25</wheel_normal_force>
+      </wheel>
+      <wheel link_name="wheel2">
+        <slip_compliance_lateral>0.05</slip_compliance_lateral>
+        <slip_compliance_longitudinal>0.0</slip_compliance_longitudinal>
+        <wheel_normal_force>25</wheel_normal_force>
+      </wheel>
+      <wheel link_name="wheel3">
+        <slip_compliance_lateral>0.05</slip_compliance_lateral>
+        <slip_compliance_longitudinal>0.0</slip_compliance_longitudinal>
+        <wheel_normal_force>25</wheel_normal_force>
+      </wheel>
+    </plugin>
+  </gazebo>
 </robot>

Commit message: fixed timing issues for controllers loading

File: src/my_robot_description/urdf/robot_v3.xacro (robot description, xacro)
@@ -906,95 +906,53 @@
   </gazebo>
   <gazebo reference="lidarView">
-      <sensor name="lidarView" type="gpu_lidar">
-          <pose>0 0 0 0 0 0</pose>
-          <topic>lidar</topic>
-          <update_rate>20</update_rate>
-          <ray>
-            <scan>
-              <horizontal>
-                <samples>360</samples>
-                <resolution>1</resolution>
-                <min_angle>-3.14159</min_angle>
-                <max_angle>3.14159</max_angle>
-              </horizontal>
-              <vertical>
-                <samples>1</samples>
-                <resolution>1</resolution>
-                <min_angle>0</min_angle>
-                <max_angle>0</max_angle>
-              </vertical>
-            </scan>
-            <range>
-              <min>0.12</min>
-              <max>6.0</max>
-              <resolution>0.01</resolution>
-            </range>
-          </ray>
-          <always_on>1</always_on>
-          <visualize>true</visualize>
-        </sensor>
+      <sensor name="lidarView" type="gpu_lidar">  <!-- Changed from gpu_lidar to regular lidar -->
+        <pose>0 0 0 0 0 0</pose>
+        <topic>/scan</topic>
+        <ignition_frame_id>lidarView</ignition_frame_id>
+        <update_rate>10</update_rate>  <!-- Reduced from 20 to 10 Hz -->
+        <ray>
+          <scan>
+            <horizontal>
+              <samples>180</samples>  <!-- Reduced from 360 to 180 samples -->
+              <resolution>1</resolution>
+              <min_angle>-3.14159</min_angle>  <!-- -90 degrees instead of full circle -->
+              <max_angle>3.14159</max_angle>   <!-- +90 degrees -->
+            </horizontal>
+            <vertical>
+              <samples>1</samples>
+              <resolution>1</resolution>
+              <min_angle>0</min_angle>
+              <max_angle>0</max_angle>
+            </vertical>
+          </scan>
+          <range>
+            <min>0.12</min>
+            <max>4.0</max>  <!-- Reduced from 6.0 to 4.0 meters -->
+            <resolution>0.05</resolution>  <!-- Reduced resolution from 0.01 to 0.05 -->
+          </range>
+        </ray>
+        <always_on>1</always_on>
+        <visualize>false</visualize>
+    </sensor>
   </gazebo>
-  <!-- URDF file -->
-  <link name="imu_link">
-    <inertial><mass value="1e-6"/></inertial>
-  </link>
+  <!-- IMU frame: no inertial on sensor link -->
+  <link name="imu_link"/>
   <joint name="imu_joint" type="fixed">
     <parent link="base_link"/>
-    <child link="imu_link"/>
+    <child  link="imu_link"/>
     <origin xyz="0 0 0.10" rpy="0 0 0"/>
   </joint>
-  <!-- SDF-in-URDF block that Gazebo reads -->
+  <!-- Ignition/GZ reads <gazebo> tags embedded in URDF -->
   <gazebo reference="imu_link">
     <sensor name="imu" type="imu">
-      <always_on>1</always_on>
-      <update_rate>100</update_rate>
+      <always_on>true</always_on>
+      <update_rate>50</update_rate>  <!-- Reduced from 100 to 50 Hz -->
       <visualize>false</visualize>
-      <!-- Gazebo transport topic name; ros_gz_bridge will bridge this to ROS -->
       <topic>imu</topic>
-      <!-- Frame id for ROS (supported by ros_gz); harmless warning if not recognized) -->
-      <gz_frame_id>imu_link</gz_frame_id>
-      <!-- Optional: add noise (example values) -->
+      <ignition_frame_id>imu_link</ignition_frame_id>
       <imu>
+        <!-- leave empty for ideal IMU in sim -->
       </imu>
     </sensor>
   </gazebo>
-    <!-- wheel1 -->
-  <gazebo reference="wheel1">
-    <mu1>1.6</mu1>
-    <mu2>0.01</mu2>
-    <!-- Try +X of wheel1 as rolling dir first -->
-    <fdir1 gz:expressed_in="wheel1">1 0 0</fdir1>
-  </gazebo>
-  <!-- wheel2 -->
-  <gazebo reference="wheel2">
-    <mu1>1.6</mu1>
-    <mu2>0.01</mu2>
-    <fdir1 gz:expressed_in="wheel2">0 1 0</fdir1>
-  </gazebo>
-  <!-- wheel3 -->
-  <gazebo reference="wheel3">
-    <mu1>1.6</mu1>
-    <mu2>0.01</mu2>
-    <fdir1 gz:expressed_in="wheel3">-1 0 0</fdir1>
-  </gazebo>
-  <gazebo>
-    <plugin name="ignition::gazebo::systems::WheelSlip"
-            filename="libignition-gazebo-wheel-slip-system.so">
-      <wheel link_name="wheel1">
-        <slip_compliance_lateral>0.05</slip_compliance_lateral>
-        <slip_compliance_longitudinal>0.0</slip_compliance_longitudinal>
-        <wheel_normal_force>25</wheel_normal_force>
-      </wheel>
-      <wheel link_name="wheel2">
-        <slip_compliance_lateral>0.05</slip_compliance_lateral>
-        <slip_compliance_longitudinal>0.0</slip_compliance_longitudinal>
-        <wheel_normal_force>25</wheel_normal_force>
-      </wheel>
-      <wheel link_name="wheel3">
-        <slip_compliance_lateral>0.05</slip_compliance_lateral>
-        <slip_compliance_longitudinal>0.0</slip_compliance_longitudinal>
-        <wheel_normal_force>25</wheel_normal_force>
-      </wheel>
-    </plugin>
-  </gazebo>
 </robot>

Commit message: fixed slam config and omni geometery and odometry

File: src/my_robot_description/urdf/robot_v3.xacro (robot description, xacro)
@@ -765,12 +765,4 @@
         <mesh filename="file://$(find my_robot_description)/models/delivery_bot/meshes/wheel.stl"/>
       </geometry>
-      <surface>
-        <friction>
-          <ode>
-            <mu>1.0</mu>
-            <mu2>1.0</mu2>
-          </ode>
-        </friction>
-      </surface>
     </collision>
   </link>
@@ -778,4 +770,5 @@
   <joint name="wheel1_joint" type="continuous">
     <origin xyz="-0.100026 0.05775 -0.0195" rpy="1.5708 1.48832 1.0472"/>
+    <!-- 1.48832 -->
     <parent link="base_link"/>
     <child link="wheel1"/>
@@ -783,7 +776,7 @@
     <axis xyz="0 0 1"/>
     <!-- Continuous joints ignore lower/upper. Keep effort/velocity. -->
-    <limit effort="5.0" velocity="100.0"/>
+    <limit effort="15.0" velocity="100.0"/>
     <!-- Helps kill jitter -->
-    <dynamics damping="0.2" friction="0.0"/>
+    <dynamics damping="0.1" friction="0.05"/>
   </joint>
   <!-- Link wheel2 -->
@@ -809,12 +802,4 @@
         <mesh filename="file://$(find my_robot_description)/models/delivery_bot/meshes/wheel.stl"/>
       </geometry>
-      <surface>
-        <friction>
-          <ode>
-            <mu>1.0</mu>
-            <mu2>1.0</mu2>
-          </ode>
-        </friction>
-      </surface>
     </collision>
   </link>  <!-- wheel2: make it continuous and remove position limits -->
@@ -826,7 +811,7 @@
     <axis xyz="0 0 1"/>
     <!-- Continuous joints ignore lower/upper. Keep effort/velocity. -->
-    <limit effort="5.0" velocity="100.0"/>
+    <limit effort="15.0" velocity="100.0"/>
     <!-- Helps kill jitter -->
-    <dynamics damping="0.2" friction="0.0"/>
+    <dynamics damping="0.1" friction="0.05"/>
   </joint>
   <!-- Link wheel3 -->
@@ -852,12 +837,4 @@
         <mesh filename="file://$(find my_robot_description)/models/delivery_bot/meshes/wheel.stl"/>
       </geometry>
-      <surface>
-        <friction>
-          <ode>
-            <mu>1.0</mu>
-            <mu2>1.0</mu2>
-          </ode>
-        </friction>
-      </surface>
     </collision>
   </link>
@@ -871,8 +848,50 @@
     <axis xyz="0 0 1"/>
     <!-- Continuous joints ignore lower/upper. Keep effort/velocity. -->
-    <limit effort="5.0" velocity="100.0"/>
+    <limit effort="15.0" velocity="100.0"/>
     <!-- Helps kill jitter -->
-    <dynamics damping="0.2" friction="0.0"/>
+    <dynamics damping="0.1" friction="0.05"/>
   </joint>
+  <!-- Gazebo properties for wheel1 -->
+  <gazebo reference="wheel1">
+    <surface>
+      <friction>
+        <ode>
+          <mu>0.1</mu>      <!-- Rolling direction -->
+          <mu2>1.0</mu2>    <!-- Perpendicular direction -->
+          <slip1>0.0</slip1>
+          <slip2>1.0</slip2>
+        </ode>
+      </friction>
+    </surface>
+    <material>Gazebo/Blue</material>
+  </gazebo>
+  <!-- Gazebo properties for wheel2 -->
+  <gazebo reference="wheel2">
+    <surface>
+      <friction>
+        <ode>
+          <mu>0.1</mu>      <!-- Rolling direction -->
+          <mu2>1.0</mu2>    <!-- Perpendicular direction -->
+          <slip1>0.0</slip1>
+          <slip2>1.0</slip2>
+        </ode>
+      </friction>
+    </surface>
+    <material>Gazebo/Blue</material>
+  </gazebo>
+  <!-- Gazebo properties for wheel3 -->
+  <gazebo reference="wheel3">
+    <surface>
+      <friction>
+        <ode>
+          <mu>0.1</mu>      <!-- Rolling direction -->
+          <mu2>1.0</mu2>    <!-- Perpendicular direction -->
+          <slip1>0.0</slip1>
+          <slip2>1.0</slip2>
+        </ode>
+      </friction>
+    </surface>
+    <material>Gazebo/Blue</material>
+  </gazebo>
   <!-- ROS2 Control for Fortress -->
   <ros2_control name="GazeboSimSystem" type="system">
@@ -910,9 +929,9 @@
       <topic>/scan</topic>
       <gz_frame_id>lidarView</gz_frame_id>
-      <update_rate>10</update_rate>  <!-- Reduced from 20 to 10 Hz -->
+      <update_rate>25</update_rate>  <!-- Reduced from 20 to 10 Hz -->
       <ray>
         <scan>
           <horizontal>
-            <samples>180</samples>  <!-- Reduced from 360 to 180 samples -->
+            <samples>360</samples>  <!-- Reduced from 360 to 180 samples -->
             <resolution>1</resolution>
             <min_angle>-3.14159</min_angle>  <!-- -90 degrees instead of full circle -->
