Commit message: switched to harmonic and jazzy and used official omni wheel controller instead of custom nodes

File: src/my_robot_description/urdf/robot_v3.xacro (robot description, xacro)
@@ -743,32 +743,30 @@
     <axis xyz="0 0 0"/>
   </joint>
-  <!-- Link wheel -->
+  <!-- Link wheel1 -->
   <link name="wheel1">
     <inertial>
-      <origin xyz="4.50126e-19 -6.90649e-18 -0.0125" rpy="0 0 0"/>
+      <origin xyz="6.66143e-18 1.48071e-18 -0.0125" rpy="0 0 0"/>
       <mass value="0.056156"/>
-      <inertia ixx="1.10674e-05" ixy="-1.53591e-22" ixz="-1.26001e-22" iyy="1.10674e-05" iyz="8.14835e-22" izz="1.62852e-05"/>
+      <inertia ixx="1.10674e-05" ixy="-1.51453e-52" ixz="-2.89647e-22" iyy="1.10674e-05" iyz="-5.04438e-69" izz="1.62852e-05"/>
     </inertial>
-    <!-- Part wheel -->
-    <visual>
-      <origin xyz="0 -8.67362e-18 -0.025" rpy="3.99084e-17 6.27965e-18 -1.38778e-17"/>
+    <!-- Part wheel2 -->
+    <visual>
+      <origin xyz="6.86182e-18 0 -0.025" rpy="0 -5.55112e-17 -8.21073e-48"/>
       <geometry>
         <mesh filename="file://$(find my_robot_description)/models/delivery_bot/meshes/wheel.stl"/>
       </geometry>
-      <material name="wheel_material">
-        <color rgba="0.615686 0.811765 0.929412 1"/>
-      </material>
-    </visual>
-    <collision>
-      <origin xyz="0 -8.67362e-18 -0.025" rpy="3.99084e-17 6.27965e-18 -1.38778e-17"/>
+      <material name="wheel2_material">
+        <color rgba="0.615686 0.811765 0.929412 1"/>
+      </material>
+    </visual>
+    <collision>
+      <origin xyz="6.86182e-18 0 -0.025" rpy="0 -5.55112e-17 -8.21073e-48"/>
       <geometry>
         <mesh filename="file://$(find my_robot_description)/models/delivery_bot/meshes/wheel.stl"/>
       </geometry>
     </collision>
-  </link>
-  <!-- wheel1: make it continuous and remove position limits -->
+  </link>  <!-- wheel1: make it continuous and remove position limits -->
   <joint name="wheel1_joint" type="continuous">
-    <origin xyz="-0.100026 0.05775 -0.0195" rpy="1.5708 1.48832 1.0472"/>
-    <!-- 1.48832 -->
+    <origin xyz="0.100026 0.05775 -0.0195" rpy="1.5708 -2.15704e-32 -1.0472"/>
     <parent link="base_link"/>
     <child link="wheel1"/>
@@ -783,27 +781,29 @@
   <link name="wheel2">
     <inertial>
-      <origin xyz="6.66143e-18 1.48071e-18 -0.0125" rpy="0 0 0"/>
+      <origin xyz="4.50126e-19 -6.90649e-18 -0.0125" rpy="0 0 0"/>
       <mass value="0.056156"/>
-      <inertia ixx="1.10674e-05" ixy="-1.51453e-52" ixz="-2.89647e-22" iyy="1.10674e-05" iyz="-5.04438e-69" izz="1.62852e-05"/>
+      <inertia ixx="1.10674e-05" ixy="-1.53591e-22" ixz="-1.26001e-22" iyy="1.10674e-05" iyz="8.14835e-22" izz="1.62852e-05"/>
     </inertial>
     <!-- Part wheel2 -->
     <visual>
-      <origin xyz="6.86182e-18 0 -0.025" rpy="0 -5.55112e-17 -8.21073e-48"/>
+      <origin xyz="0 -8.67362e-18 -0.025" rpy="3.99084e-17 6.27965e-18 -1.38778e-17"/>
       <geometry>
         <mesh filename="file://$(find my_robot_description)/models/delivery_bot/meshes/wheel.stl"/>
       </geometry>
-      <material name="wheel2_material">
-        <color rgba="0.615686 0.811765 0.929412 1"/>
-      </material>
-    </visual>
-    <collision>
-      <origin xyz="6.86182e-18 0 -0.025" rpy="0 -5.55112e-17 -8.21073e-48"/>
+      <material name="wheel_material">
+        <color rgba="0.615686 0.811765 0.929412 1"/>
+      </material>
+    </visual>
+    <collision>
+      <origin xyz="0 -8.67362e-18 -0.025" rpy="3.99084e-17 6.27965e-18 -1.38778e-17"/>
       <geometry>
         <mesh filename="file://$(find my_robot_description)/models/delivery_bot/meshes/wheel.stl"/>
       </geometry>
     </collision>
-  </link>  <!-- wheel2: make it continuous and remove position limits -->
+  </link>
+  <!-- wheel2: make it continuous and remove position limits -->
   <joint name="wheel2_joint" type="continuous">
-    <origin xyz="0.100026 0.05775 -0.0195" rpy="1.5708 -2.15704e-32 -1.0472"/>
+    <origin xyz="-0.100026 0.05775 -0.0195" rpy="1.5708 1.48832 1.0472"/>
+    <!-- 1.48832 -->
     <parent link="base_link"/>
     <child link="wheel2"/>
@@ -854,48 +854,54 @@
   <!-- Gazebo properties for wheel1 -->
   <gazebo reference="wheel1">
-    <surface>
-      <friction>
-        <ode>
-          <mu>0.1</mu>      <!-- Rolling direction -->
-          <mu2>1.0</mu2>    <!-- Perpendicular direction -->
-          <slip1>0.0</slip1>
-          <slip2>1.0</slip2>
-        </ode>
-      </friction>
-    </surface>
+    <collision>
+      <surface>
+        <friction>
+          <ode>
+            <mu>5.0</mu>
+            <mu2>0.001</mu2>
+            <slip1>0.0</slip1>
+            <slip2>5.0</slip2>
+          </ode>
+        </friction>
+      </surface>
+    </collision>
     <material>Gazebo/Blue</material>
   </gazebo>
   <!-- Gazebo properties for wheel2 -->
   <gazebo reference="wheel2">
-    <surface>
-      <friction>
-        <ode>
-          <mu>0.1</mu>      <!-- Rolling direction -->
-          <mu2>1.0</mu2>    <!-- Perpendicular direction -->
-          <slip1>0.0</slip1>
-          <slip2>1.0</slip2>
-        </ode>
-      </friction>
-    </surface>
+    <collision>
+      <surface>
+        <friction>
+          <ode>
+            <mu>5.0</mu>
+            <mu2>0.001</mu2>
+            <slip1>0.0</slip1>
+            <slip2>5.0</slip2>
+          </ode>
+        </friction>
+      </surface>
+    </collision>
     <material>Gazebo/Blue</material>
   </gazebo>
   <!-- Gazebo properties for wheel3 -->
   <gazebo reference="wheel3">
-    <surface>
-      <friction>
-        <ode>
-          <mu>0.1</mu>      <!-- Rolling direction -->
-          <mu2>1.0</mu2>    <!-- Perpendicular direction -->
-          <slip1>0.0</slip1>
-          <slip2>1.0</slip2>
-        </ode>
-      </friction>
-    </surface>
+    <collision>
+      <surface>
+        <friction>
+          <ode>
+            <mu>5.0</mu>
+            <mu2>0.001</mu2>
+            <slip1>0.0</slip1>
+            <slip2>5.0</slip2>
+          </ode>
+        </friction>
+      </surface>
+    </collision>
     <material>Gazebo/Blue</material>
   </gazebo>
-  <!-- ROS2 Control for Fortress -->
+  <!-- ROS2 Control for Harmonic - UPDATED -->
   <ros2_control name="GazeboSimSystem" type="system">
     <hardware>
-      <plugin>gz_ros2_control/GazeboSimSystem</plugin>
+      <plugin>gz_ros2_control/GazeboSimSystem</plugin>  <!-- Updated plugin name -->
     </hardware>
     <joint name="wheel1_joint">
@@ -915,42 +921,40 @@
     </joint>
   </ros2_control>
-  <!-- Gazebo ROS2 Control Plugin for Fortress -->
+  <!-- Gazebo ROS2 Control Plugin for Harmonic - MAJOR CHANGES -->
   <gazebo>
-    <plugin filename="libign_ros2_control-system.so"
-            name="ign_ros2_control::IgnitionROS2ControlPlugin">
+     <plugin filename="libgz_ros2_control-system.so" name="gz_ros2_control::GazeboSimROS2ControlPlugin">
       <robot_param>robot_description</robot_param>
       <robot_param_node>robot_state_publisher</robot_param_node>
-      <parameters>/home/abanoub/delivery_bot_ws/src/delivery_bot_control/config/omni_drive_controller.params.yaml</parameters>
+      <parameters>/home/abanoub/delivery_bot_ws/src/delivery_bot_control/config/omni_drive_controller.yaml</parameters>
     </plugin>
   </gazebo>
+  <!-- LiDAR sensor - CORRECTED for Gazebo Harmonic -->
   <gazebo reference="lidarView">
     <sensor name="lidarView" type="gpu_lidar">
-      <pose>0 0 0 0 0 0</pose>
+      <gz_frame_id>lidarView</gz_frame_id>
+      <always_on>true</always_on>
+      <update_rate>20</update_rate>
+      <visualize>false</visualize>
       <topic>/scan</topic>
-      <gz_frame_id>lidarView</gz_frame_id>
-      <update_rate>25</update_rate>  <!-- Reduced from 20 to 10 Hz -->
-      <ray>
+      <plugin filename="libgz-sim-sensors-system.so" name="gz::sim::systems::Sensors">
+        <render_engine>ogre2</render_engine>
+      </plugin>
+      <pose relative_to="lidarView">0 0 0 0 0 0</pose>
+      <!-- plugin already included in world file -->
+      <lidar>
         <scan>
           <horizontal>
-            <samples>360</samples>  <!-- Reduced from 360 to 180 samples -->
+            <samples>360</samples>
             <resolution>1</resolution>
-            <min_angle>-3.14159</min_angle>  <!-- -90 degrees instead of full circle -->
-            <max_angle>3.14159</max_angle>   <!-- +90 degrees -->
+            <min_angle>-3.14</min_angle>
+            <max_angle>3.14</max_angle>
           </horizontal>
-          <vertical>
-            <samples>1</samples>
-            <resolution>1</resolution>
-            <min_angle>0</min_angle>
-            <max_angle>0</max_angle>
-          </vertical>
         </scan>
         <range>
           <min>0.12</min>
           <max>6.0</max>
-          <resolution>0.05</resolution>  <!-- Reduced resolution from 0.01 to 0.05 -->
+          <resolution>0.05</resolution>
         </range>
-      </ray>
-      <always_on>1</always_on>
-      <visualize>false</visualize>
+      </lidar>
     </sensor>
   </gazebo>
@@ -962,14 +966,53 @@
     <origin xyz="0 0 0.10" rpy="0 0 0"/>
   </joint>
-  <!-- Ignition/GZ reads <gazebo> tags embedded in URDF -->
+  <!-- IMU sensor - CORRECTED for Gazebo Harmonic -->
   <gazebo reference="imu_link">
     <sensor name="imu" type="imu">
+      <gz_frame_id>imu_link</gz_frame_id>
       <always_on>true</always_on>
-      <update_rate>50</update_rate>  <!-- Reduced from 100 to 50 Hz -->
+      <update_rate>50.0</update_rate>
       <visualize>false</visualize>
-      <topic>imu</topic>
-      <gz_frame_id>imu_link</gz_frame_id>
+      <topic>/imu</topic>
       <imu>
-        <!-- leave empty for ideal IMU in sim -->
+        <angular_velocity>
+          <x>
+            <noise type="gaussian">
+              <mean>0.0</mean>
+              <stddev>2e-4</stddev>
+            </noise>
+          </x>
+          <y>
+            <noise type="gaussian">
+              <mean>0.0</mean>
+              <stddev>2e-4</stddev>
+            </noise>
+          </y>
+          <z>
+            <noise type="gaussian">
+              <mean>0.0</mean>
+              <stddev>2e-4</stddev>
+            </noise>
+          </z>
+        </angular_velocity>
+        <linear_acceleration>
+          <x>
+            <noise type="gaussian">
+              <mean>0.0</mean>
+              <stddev>1.7e-2</stddev>
+            </noise>
+          </x>
+          <y>
+            <noise type="gaussian">
+              <mean>0.0</mean>
+              <stddev>1.7e-2</stddev>
+            </noise>
+          </y>
+          <z>
+            <noise type="gaussian">
+              <mean>0.0</mean>
+              <stddev>1.7e-2</stddev>
+            </noise>
+          </z>
+        </linear_acceleration>
       </imu>
     </sensor>

Commit message: changed maze and slam settings to allow for loop closure for cleaner SLAM also fixed sign convention of wheel_odom to match imu

File: src/my_robot_description/urdf/robot_v3.xacro (robot description, xacro)
@@ -772,5 +772,5 @@
     <child link="wheel1"/>
     <!-- Axis must be the wheel's spin axis in the JOINT frame -->
-    <axis xyz="0 0 1"/>
+    <axis xyz="0 0 -1"/>
     <!-- Continuous joints ignore lower/upper. Keep effort/velocity. -->
     <limit effort="15.0" velocity="100.0"/>
@@ -809,5 +809,5 @@
     <child link="wheel2"/>
     <!-- Axis must be the wheel's spin axis in the JOINT frame -->
-    <axis xyz="0 0 1"/>
+    <axis xyz="0 0 -1"/>
     <!-- Continuous joints ignore lower/upper. Keep effort/velocity. -->
     <limit effort="15.0" velocity="100.0"/>
@@ -846,5 +846,5 @@
     <child link="wheel3"/>
     <!-- Axis must be the wheel's spin axis in the JOINT frame -->
-    <axis xyz="0 0 1"/>
+    <axis xyz="0 0 -1"/>
     <!-- Continuous joints ignore lower/upper. Keep effort/velocity. -->
     <limit effort="15.0" velocity="100.0"/>
@@ -907,5 +907,5 @@
       <gz_frame_id>lidarView</gz_frame_id>
       <always_on>true</always_on>
-      <update_rate>20</update_rate>
+      <update_rate>25</update_rate>
       <visualize>false</visualize>
       <topic>/scan</topic>
@@ -944,5 +944,5 @@
       <gz_frame_id>imu_link</gz_frame_id>
       <always_on>true</always_on>
-      <update_rate>50.0</update_rate>
+      <update_rate>100.0</update_rate>
       <visualize>false</visualize>
       <topic>/imu</topic>
